File: sensor-hub.kicad_pcb (KiCad board)
At the start: 2 copper layers, 91.4 x 71.1 mm, 21 parts, among them J1 Barrel_Jack_Switch, J2 Screw_Terminal_01x08, SW1 SW_SPDT, SW2 SW_SPST, U1 MCP23017_SP, U2 MCP1700x-500xxTO

Commit message: v1 ready with a perfboard placement in pcb editor planned out
Parts:
- removed C1, C2: 1u, Capacitor_THT:CP_Radial_D10.0mm_P2.50mm
- removed U2: MCP1700x-500xxTO, Package_TO_SOT_THT:TO-92_Inline
- added BZ1: Buzzer, Buzzer_Beeper:Buzzer_12x9.5RM7.6, F.Cu at (109.2, 113.0)
- added D4: LED, LED_THT:LED_D3.0mm, F.Cu at (185.4, 91.4)
- added D5: LED, LED_THT:LED_D3.0mm, F.Cu at (165.1, 154.9)
- added J3: 01x01_Pin, Connector_PinHeader_1.00mm:PinHeader_1x01_P1.00mm_Vertical, F.Cu at (188.0, 137.2)
- added J4: 01x01_Pin, Connector_PinHeader_1.00mm:PinHeader_1x01_P1.00mm_Vertical, F.Cu at (170.2, 96.5)
- added J5: 01x01_Pin, Connector_PinHeader_1.00mm:PinHeader_1x01_P1.00mm_Vertical, F.Cu at (170.2, 137.2)
- added J6: 01x01_Pin, Connector_PinHeader_1.00mm:PinHeader_1x01_P1.00mm_Vertical, F.Cu at (188.0, 96.5)
- added Q2: NPN, Package_TO_SOT_THT:TO-92, F.Cu at (119.4, 105.4)
- added R10: 4,7k, Resistor_THT:R_Axial_DIN0207_L6.3mm_D2.5mm_P2.54mm_Vertical, F.Cu at (132.1, 134.6)
- added R11: 4,7k, Resistor_THT:R_Axial_DIN0207_L6.3mm_D2.5mm_P2.54mm_Vertical, F.Cu at (127.0, 134.6)
- added R9: 1k, Resistor_THT:R_Axial_DIN0207_L6.3mm_D2.5mm_P2.54mm_Vertical, F.Cu at (129.5, 106.7)
- C3: value 0.1u -> 0,1u; footprint Capacitor_THT:CP_Radial_D10.0mm_P2.50mm -> Capacitor_THT:C_Disc_D5.0mm_W2.5mm_P5.00mm
- R3, R4: value 10k -> 1k
- R7: value 20k -> 1k
- moved D1 193.5 mm to (162.6, 116.8), turned to 90 degrees
- moved D2 124.3 mm to (99.0, 75.8)
- moved D3 124.3 mm to (94.0, 76.2)
- moved C3 94.9 mm to (165.1, 94.0), turned to 90 degrees
- moved R7 50.8 mm to (172.7, 91.4)
- moved R4 48.9 mm to (165.1, 144.8), turned to -90 degrees
- moved U1 38.9 mm to (121.9, 152.4), turned to 180 degrees
- moved R5 38.8 mm to (132.1, 116.8)
- moved R1 33.1 mm to (154.9, 99.1), turned to 180 degrees
- moved R8 30.6 mm to (162.6, 101.6), turned to -90 degrees
- moved R2 27.9 mm to (160.0, 96.5), turned to 90 degrees
- moved J1 11.2 mm to (174.3, 146.4), turned to 90 degrees
- moved R3 5.68 mm to (144.8, 99.1), turned to 0 degrees
- moved SW1 2.54 mm to (149.9, 91.4)
Connections:
- A1 pad 21: unconnected-(A1-GPIO16-Pad21) -> /BUZZER
- A1 pad 25: unconnected-(A1-GPIO19-Pad25) -> /MCP_RESET
- A1 pad 27: unconnected-(A1-GPIO21-Pad27) -> /INTA
- A1 pad 30: unconnected-(A1-RUN-Pad30) -> /PICO_RUN
- A1 pad 31: unconnected-(A1-GPIO26_ADC0-Pad31) -> /SDA
- A1 pad 32: unconnected-(A1-GPIO27_ADC1-Pad32) -> /SCK
- A1 pad 39: +5V -> /+5V_A
- A1 pad 4: /INTA -> unconnected-(A1-GPIO2-Pad4)
- A1 pad 5: Net-(A1-GPIO3) -> /ARM_DISARM
- D1 pad 1: +5V -> /+5V_A
- D1 pad 2: Net-(D1-A) -> /+5V_A_PRES
- R1 pad 1: +5V -> +3.3V
- R3 pad 1: +5V -> Net-(SW1-B)
- R3 pad 2: Net-(SW1-C) -> /ARM_DISARM
- R4 pad 1: Net-(SW1-C) -> /VIN_RAW
- R4 pad 2: Net-(R4-Pad2) -> Net-(D5-A)
- R5 pad 1: GND -> /MCP_RESET
- R5 pad 2: Net-(R4-Pad2) -> +3.3V
- R7 pad 1: GND -> /+5V_A_PRES
- R7 pad 2: Net-(SW2-B) -> Net-(D4-A)
- SW1 pad 2: Net-(A1-GPIO3) -> Net-(SW1-B)
- SW1 pad 3: Net-(SW1-C) -> +3.3V
- U1 pad 18: +5V -> /MCP_RESET
- U1 pad 9: +5V -> +3.3V
Routing:
- net GND: track 0.00 -> 232.1 mm
- net +3.3V: track 0.00 -> 115.8 mm
- net /+5V_A: track 0.00 -> 106.3 mm
- net Net-(SW2-B): track 0.00 -> 68.9 mm
- net /ARM_DISARM: track 0.00 -> 49.4 mm
- net /RESET_SW: track 0.00 -> 40.7 mm
- net /MCP_RESET: track 0.00 -> 29.3 mm
- net /INTA: track 0.00 -> 28.3 mm
- net /+5V_A_PRES: track 0.00 -> 27.1 mm
- net /SCK: track 0.00 -> 20.7 mm
- net /A0_IN: track 0.00 -> 12.3 mm
- net /A1_IN: track 0.00 -> 11.9 mm
- net /A2_IN: track 0.00 -> 11.5 mm
- net /SDA: track 0.00 -> 11.4 mm
- net /A3_IN: track 0.00 -> 11.1 mm
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